Commit message: try to add world

File: simple_robot_description/urdf/simple_robot.xacro (robot description, xacro)
@@ -104,5 +104,5 @@
   </collision>
 </link>
-<joint name="Rev1" type="continuous">
+<joint name="base_link_left_wheel_joint" type="continuous">
   <origin rpy="0 0 0" xyz="0.0 0.1 0.075"/>
   <parent link="base_link"/>
@@ -110,5 +110,5 @@
   <axis xyz="0.0 1.0 0.0"/>
 </joint>
-<joint name="Rev2" type="continuous">
+<joint name="base_link_right_wheel_joint" type="continuous">
   <origin rpy="0 0 0" xyz="0.0 -0.1 0.075"/>
   <parent link="base_link"/>

Commit message: no errors

File: simple_robot_description/urdf/simple_robot.xacro (robot description, xacro)
@@ -104,5 +104,5 @@
   </collision>
 </link>
-<joint name="base_link_left_wheel_joint" type="continuous">
+<joint name="Rev1" type="continuous">
   <origin rpy="0 0 0" xyz="0.0 0.1 0.075"/>
   <parent link="base_link"/>
@@ -110,5 +110,5 @@
   <axis xyz="0.0 1.0 0.0"/>
 </joint>
-<joint name="base_link_right_wheel_joint" type="continuous">
+<joint name="Rev2" type="continuous">
   <origin rpy="0 0 0" xyz="0.0 -0.1 0.075"/>
   <parent link="base_link"/>

Commit message: add gmapping to real robot

File: simple_robot_description/urdf/simple_robot.xacro (robot description, xacro)
@@ -64,5 +64,5 @@
   </collision>
 </link>
-<link name="lidar_1">
+<link name="laser">
   <inertial>
     <origin rpy="0 0 0" xyz="0.0 9.046911093940672e-18 0.024999999999999994"/>
@@ -119,5 +119,5 @@
   <origin rpy="0 0 0" xyz="0.01 0.0 0.165"/>
   <parent link="base_link"/>
-  <child link="lidar_1"/>
+  <child link="laser"/>
 </joint>
 <joint name="Rigid4" type="fixed">
