Commit message: add imu to robot

File: simple_robot/simple_robot_description/urdf/simple.urdf.xacro (robot description, xacro)
@@ -43,4 +43,11 @@
     <gravity>true</gravity>
   </gazebo>
+  <link name="imu_link">
+  </link>
+  <joint name="base_to_imu" type="fixed">
+    <parent link="base_link"/>
+    <child link="imu_link"/>
+    <origin rpy="0 0 0" xyz="0 0 0"/>
+  </joint>
   <link name="caster_wheel">
     <visual>
@@ -119,3 +126,23 @@
     </plugin>
   </gazebo>
+  <gazebo reference="imu_link">
+    <gravity>true</gravity>
+    <sensor name="imu_sensor" type="imu">
+      <always_on>true</always_on>
+      <update_rate>100</update_rate>
+      <visualize>true</visualize>
+      <topic>__default_topic__</topic>
+      <plugin filename="libgazebo_ros_imu_sensor.so" name="imu_plugin">
+        <topicName>imu</topicName>
+        <bodyName>imu_link</bodyName>
+        <updateRateHZ>10.0</updateRateHZ>
+        <gaussianNoise>0.0</gaussianNoise>
+        <xyzOffset>0 0 0</xyzOffset>
+        <rpyOffset>0 0 0</rpyOffset>
+        <frameName>imu_link</frameName>
+        <initialOrientationAsReference>false</initialOrientationAsReference>
+      </plugin>
+      <pose>0 0 0 0 0 0</pose>
+    </sensor>
+  </gazebo>
 </robot>

Commit message: added imu working

File: simple_robot/simple_robot_description/urdf/simple.urdf.xacro (robot description, xacro)
@@ -43,4 +43,11 @@
     <gravity>true</gravity>
   </gazebo>
+  <link name="imu_link">
+  </link>
+  <joint name="base_to_imu" type="fixed">
+    <parent link="base_link"/>
+    <child link="imu_link"/>
+    <origin rpy="0 0 0" xyz="0 0 ${wheel_dia/2+hight/2}"/>
+  </joint>
   <link name="caster_wheel">
     <visual>
@@ -119,3 +126,24 @@
     </plugin>
   </gazebo>
+  <!-- imu  -->
+  <gazebo reference="imu_link">
+    <gravity>true</gravity>
+    <sensor name="imu_sensor" type="imu">
+      <always_on>true</always_on>
+      <update_rate>100</update_rate>
+      <visualize>true</visualize>
+      <topic>__default_topic__</topic>
+      <plugin filename="libgazebo_ros_imu_sensor.so" name="imu_plugin">
+        <topicName>imu</topicName>
+        <bodyName>imu_link</bodyName>
+        <updateRateHZ>10.0</updateRateHZ>
+        <gaussianNoise>0.0</gaussianNoise>
+        <xyzOffset>0 0 0</xyzOffset>
+        <rpyOffset>0 0 0</rpyOffset>
+        <frameName>imu_link</frameName>
+        <initialOrientationAsReference>false</initialOrientationAsReference>
+      </plugin>
+      <pose>0 0 0 0 0 0</pose>
+    </sensor>
+  </gazebo>
 </robot>

Commit message: add lidar

File: simple_robot/simple_robot_description/urdf/simple.urdf.xacro (robot description, xacro)
@@ -3,9 +3,11 @@
   <xacro:property name="width" value="0.18" />
   <xacro:property name="length" value="0.25" />
-  <xacro:property name="hight" value="0.2" />
+  <xacro:property name="height" value="0.2" />
   <xacro:property name="caster_dia" value="0.02" />
   <xacro:property name="wheel_dia" value="0.064" />
   <xacro:property name="wheel_len" value="0.025" />
   <xacro:property name="wheel_separation" value="0.22" />
+  <xacro:property name="lidar_h" value="0.05" />
+  <xacro:property name="lidar_dia" value="0.07" />
   <material name="black">
     <color rgba="0 0 0 1"/>
@@ -13,4 +15,7 @@
   <material name="white">
     <color rgba="1 1 1 1"/>
+  </material>
+  <material name="blue">
+    <color rgba="0 0 1 1"/>
   </material>
   <xacro:macro name="default_inertial" params="mass">
@@ -23,19 +28,19 @@
     <visual>
       <geometry>
-        <box size="${length} ${width} ${hight}"/>
-      </geometry>
-      <origin rpy="0 0 0" xyz="0 0 ${hight/2+wheel_dia/2}"/>
+        <box size="${length} ${width} ${height}"/>
+      </geometry>
+      <origin rpy="0 0 0" xyz="0 0 ${height/2+wheel_dia/2}"/>
       <material name="white"/>
     </visual>
     <collision>
       <geometry>
-        <box size="${length} ${width} ${hight}"/>
-      </geometry>
-      <origin rpy="0 0 0" xyz="0 0 ${hight/2+wheel_dia/2}"/>
+        <box size="${length} ${width} ${height}"/>
+      </geometry>
+      <origin rpy="0 0 0" xyz="0 0 ${height/2+wheel_dia/2}"/>
     </collision>
     <xacro:default_inertial mass="20"/>
   </link>
   <gazebo reference="base_link">
-    <material>Gazebo/Blue</material>
+    <material>Gazebo/White</material>
     <mu1>0.2</mu1>
     <mu2>0.2</mu2>
@@ -48,6 +53,30 @@
     <parent link="base_link"/>
     <child link="imu_link"/>
-    <origin rpy="0 0 0" xyz="0 0 ${wheel_dia/2+hight/2}"/>
+    <origin rpy="0 0 0" xyz="0 0 ${wheel_dia/2+height/2}"/>
   </joint>
+  <link name="lidar_link">
+    <visual>
+      <geometry>
+        <cylinder length="${lidar_h}" radius="${lidar_dia/2}"/>
+      </geometry>
+      <origin rpy="0 0 0" xyz="0 0 0"/>
+      <material name="white"/>
+    </visual>
+    <collision>
+      <geometry>
+        <cylinder length="${lidar_h}" radius="${lidar_dia/2}"/>
+      </geometry>
+      <origin rpy="0 0 0" xyz="0 0 0"/>
+    </collision>
+    <xacro:default_inertial mass="20"/>
+  </link>
+  <joint name="base_to_lidar" type="fixed">
+    <parent link="base_link"/>
+    <child link="lidar_link"/>
+    <origin rpy="0 0 0" xyz="0 0 ${wheel_dia/2+height+lidar_h/2}"/>
+  </joint>
+  <gazebo reference="lidar_link">
+    <material>Gazebo/Grey</material>
+  </gazebo>
   <link name="caster_wheel">
     <visual>
@@ -147,3 +176,39 @@
     </sensor>
   </gazebo>
+  <!-- Lidar -->
+  <gazebo reference="lidar_link">
+    <sensor type="gpu_ray" name="RP_lidar">
+      <pose>0 0 0 0 0 0</pose>
+      <visualize>false</visualize>
+      <update_rate>40</update_rate>
+      <ray>
+        <scan>
+          <horizontal>
+            <samples>720</samples>
+            <resolution>1</resolution>
+            <min_angle>-3.14159</min_angle>
+            <max_angle>3.14159</max_angle>
+          </horizontal>
+        </scan>
+        <range>
+          <min>0.15</min>
+          <max>6.0</max>
+          <resolution>0.5</resolution>
+        </range>
+        <noise>
+          <type>gaussian</type>
+          <!-- Noise parameters based on published spec for Hokuyo laser
+               achieving "+-30mm" accuracy at range < 10m.  A mean of 0.0m and
+               stddev of 0.01m will put 99.7% of samples within 0.03m of the true
+               reading. -->
+          <mean>0.0</mean>
+          <stddev>0.01</stddev>
+        </noise>
+      </ray>
+      <plugin name="gazebo_ros_head_hokuyo_controller" filename="libgazebo_ros_gpu_laser.so">
+        <topicName>/scan</topicName>
+        <frameName>lidar_link</frameName>
+      </plugin>
+    </sensor>
+  </gazebo>
 </robot>

Commit message: spawn simple_robot in home

File: simple_robot/simple_robot_description/urdf/simple.urdf.xacro (robot description, xacro)
@@ -61,5 +61,5 @@
       </geometry>
       <origin rpy="0 0 0" xyz="0 0 0"/>
-      <material name="white"/>
+      <material name="black"/>
     </visual>
     <collision>
@@ -160,5 +160,5 @@
     <sensor name="imu_sensor" type="imu">
       <always_on>true</always_on>
-      <update_rate>100</update_rate>
+      <update_rate>30</update_rate>
       <visualize>true</visualize>
       <topic>__default_topic__</topic>

Commit message: ekf works in nav

File: simple_robot/simple_robot_description/urdf/simple.urdf.xacro (robot description, xacro)
@@ -10,4 +10,5 @@
   <xacro:property name="lidar_h" value="0.05" />
   <xacro:property name="lidar_dia" value="0.07" />
+  <xacro:property name="update_rate" value="30" />
   <material name="black">
     <color rgba="0 0 0 1"/>
@@ -160,5 +161,5 @@
     <sensor name="imu_sensor" type="imu">
       <always_on>true</always_on>
-      <update_rate>30</update_rate>
+      <update_rate>${update_rate}</update_rate>
       <visualize>true</visualize>
       <topic>__default_topic__</topic>
@@ -181,5 +182,5 @@
       <pose>0 0 0 0 0 0</pose>
       <visualize>false</visualize>
-      <update_rate>40</update_rate>
+      <update_rate>${update_rate}</update_rate>
       <ray>
         <scan>

Commit message: add inertia macro to urdf

File: simple_robot/simple_robot_description/urdf/simple.urdf.xacro (robot description, xacro)
@@ -20,4 +20,5 @@
     <color rgba="0 0 1 1"/>
   </material>
+  <!-- inertia -->
   <xacro:macro name="default_inertial" params="mass">
     <inertial>
@@ -26,4 +27,32 @@
     </inertial>
   </xacro:macro>
+  <xacro:macro name="box_inertial" params="m x y z">
+    <inertial>
+      <mass value="${m}" />
+      <inertia  ixx="${m*(y*y+z*z)/12}" ixy = "0" ixz = "0"
+        iyy="${m*(x*x+z*z)/12}" iyz = "0"
+        izz="${m*(x*x+z*z)/12}"
+      />
+    </inertial>
+  </xacro:macro>
+  <xacro:macro name="cylinder_inertia" params="m r h">
+    <inertial>
+      <mass value="${m}" />
+      <inertia  ixx="${m*(3*r*r+h*h)/12}" ixy = "0" ixz = "0"
+      iyy="${m*(3*r*r+h*h)/12}" iyz = "0"
+      izz="${m*r*r/2}"
+      />
+    </inertial>
+  </xacro:macro>
+  <xacro:macro name="sphere_inertia" params="m r">
+    <inertial>
+      <mass value="${m}" />
+      <inertia  ixx="${2*m*r*r/5}" ixy = "0" ixz = "0"
+        iyy="${2*m*r*r/5}" iyz = "0"
+        izz="${2*m*r*r/5}"
+      />
+    </inertial>
+  </xacro:macro>
+  <!-- base link -->
   <link name="base_link">
     <visual>
@@ -40,5 +69,5 @@
       <origin rpy="0 0 0" xyz="0 0 ${height/2+wheel_dia/2}"/>
     </collision>
-    <xacro:default_inertial mass="20"/>
+    <xacro:box_inertial m="10" x="${length}" y="${width}" z="${height}"/>
   </link>
   <gazebo reference="base_link">
@@ -49,4 +78,5 @@
     <gravity>true</gravity>
   </gazebo>
+  <!-- imu -->
   <link name="imu_link">
   </link>
@@ -56,4 +86,5 @@
     <origin rpy="0 0 0" xyz="0 0 ${wheel_dia/2+height/2}"/>
   </joint>
+  <!-- lidar -->
   <link name="lidar_link">
     <visual>
@@ -70,5 +101,5 @@
       <origin rpy="0 0 0" xyz="0 0 0"/>
     </collision>
-    <xacro:default_inertial mass="20"/>
+    <xacro:cylinder_inertia m=".3" r="${lidar_dia/2}" h="${lidar_h}"/>
   </link>
   <joint name="base_to_lidar" type="fixed">
@@ -80,4 +111,5 @@
     <material>Gazebo/Grey</material>
   </gazebo>
+  <!-- caster wheel -->
   <link name="caster_wheel">
     <visual>
@@ -94,5 +126,5 @@
       <origin rpy="0 0 0" xyz="0 0 0"/>
     </collision>
-    <xacro:default_inertial mass="0.01"/>
+   <xacro:sphere_inertia m=".01" r="${wheel_dia/2}"/>
   </link>
   <joint name="base_to_caster_wheel" type="fixed">
