Commit message: can launch turtlebot world with sr

File: simple_robot/simple_robot_description/urdf/simple_robot.urdf.xacro (robot description, xacro)
@@ -1,4 +1,5 @@
 <?xml version="1.0"?>
 <robot name="simple_robot" xmlns:xacro="http://ros.org/wiki/xacro">
+  <xacro:include filename="$(find simple_robot_description)/urdf/simple_robot.gazebo.xacro"/>
   <xacro:property name="width" value="0.18" />
   <xacro:property name="length" value="0.25" />
@@ -54,4 +55,11 @@
     </inertial>
   </xacro:macro>
+<!-- base_footprint -->
+  <link name="base_footprint"/>
+  <joint name="base_joint" type="fixed">
+    <parent link="base_footprint"/>
+    <child link="base_link"/>
+    <origin xyz="0.0 0.0 0.010" rpy="0 0 0"/>
+  </joint>
   <!-- base link -->
   <link name="base_link">
@@ -71,15 +79,7 @@
     <xacro:box_inertial m="10" x="${length}" y="${width}" z="${height}"/>
   </link>
-  <gazebo reference="base_link">
-    <material>Gazebo/White</material>
-    <mu1>0.2</mu1>
-    <mu2>0.2</mu2>
-    <selfCollide>false</selfCollide>
-    <gravity>true</gravity>
-  </gazebo>
   <!-- imu -->
-  <link name="imu_link">
-  </link>
-  <joint name="base_to_imu" type="fixed">
+  <link name="imu_link"/>
+  <joint name="imu_joint" type="fixed">
     <parent link="base_link"/>
     <child link="imu_link"/>
@@ -87,5 +87,5 @@
   </joint>
   <!-- lidar -->
-  <link name="lidar_link">
+  <link name="base_scan">
     <visual>
       <geometry>
@@ -103,10 +103,10 @@
     <xacro:cylinder_inertia m=".3" r="${lidar_dia/2}" h="${lidar_h}"/>
   </link>
-  <joint name="base_to_lidar" type="fixed">
+  <joint name="scan_joint" type="fixed">
     <parent link="base_link"/>
-    <child link="lidar_link"/>
+    <child link="base_scan"/>
     <origin rpy="0 0 0" xyz="0 0 ${wheel_dia/2+height+lidar_h/2}"/>
   </joint>
-  <gazebo reference="lidar_link">
+  <gazebo reference="base_scan">
     <material>Gazebo/Grey</material>
   </gazebo>
@@ -133,13 +133,7 @@
     <origin rpy="0 0 0" xyz="-${length/2-caster_dia/2} 0 ${wheel_dia/2}"/>
   </joint>
-  <gazebo reference="caster_wheel">
-    <mu1 value="0.0001"/>
-    <mu2 value="0.0001"/>
-    <kp value="10000000.0" />
-    <kd value="1.0" />
-    <material>Gazebo/Grey</material>
-  </gazebo>
+<!-- wheel -->
   <xacro:macro name="wheel" params="prefix reflect">
-    <link name="${prefix}_wheel">
+    <link name="wheel_${prefix}_link">
       <visual>
         <geometry>
@@ -156,18 +150,21 @@
       <xacro:default_inertial mass="0.1"/>
     </link>
-    <joint name="base_to_${prefix}_wheel" type="continuous">
+    <joint name="wheel_${prefix}_joint" type="continuous">
       <parent link="base_link"/>
-      <child link="${prefix}_wheel"/>
+      <child link="wheel_${prefix}_link"/>
       <axis xyz="0 0 -1"/>
       <origin rpy="1.5708 0 0" xyz="0.03 ${wheel_separation/2*reflect} ${wheel_dia/2}"/>
     </joint>
-    <gazebo reference="${prefix}_wheel">
-      <mu1 value="200.0"/>
-      <mu2 value="100.0"/>
-      <kp value="10000000.0" />
-      <kd value="1.0" />
-      <material>Gazebo/Grey</material>
+    <gazebo reference="wheel_${prefix}_link">
+      <mu1>0.1</mu1>
+      <mu2>0.1</mu2>
+      <kp>500000.0</kp>
+      <kd>10.0</kd>
+      <minDepth>0.001</minDepth>
+      <maxVel>0.1</maxVel>
+      <fdir1>1 0 0</fdir1>
+      <material>Gazebo/FlatBlack</material>
     </gazebo>
-    <transmission name="${prefix}_wheel_trans">
+    <!-- <transmission name="${prefix}_wheel_trans">
       <type>transmission_interface/SimpleTransmission</type>
       <actuator name="${prefix}_wheel_motor">
@@ -175,73 +172,10 @@
         <mechanicalReduction>1</mechanicalReduction>
       </actuator>
-      <joint name="base_to_${prefix}_wheel">
+      <joint name="wheel_${prefix}_joint">
         <hardwareInterface>hardware_interface/VelocityJointInterface</hardwareInterface>
       </joint>
-    </transmission>
+    </transmission> -->
   </xacro:macro>
   <xacro:wheel prefix="right" reflect="-1"/>
   <xacro:wheel prefix="left" reflect="1"/>
-  <!-- Gazebo plugin for ROS Control -->
-  <gazebo>
-    <plugin name="gazebo_ros_control" filename="libgazebo_ros_control.so">
-      <robotNamespace>/</robotNamespace>
-    </plugin>
-  </gazebo>
-  <!-- imu  -->
-  <gazebo reference="imu_link">
-    <gravity>true</gravity>
-    <sensor name="imu_sensor" type="imu">
-      <always_on>true</always_on>
-      <update_rate>${update_rate}</update_rate>
-      <visualize>true</visualize>
-      <topic>__default_topic__</topic>
-      <plugin filename="libgazebo_ros_imu_sensor.so" name="imu_plugin">
-        <topicName>imu</topicName>
-        <bodyName>imu_link</bodyName>
-        <updateRateHZ>10.0</updateRateHZ>
-        <gaussianNoise>0.01</gaussianNoise>
-        <xyzOffset>0 0 0</xyzOffset>
-        <rpyOffset>0 0 0</rpyOffset>
-        <frameName>imu_link</frameName>
-        <initialOrientationAsReference>false</initialOrientationAsReference>
-      </plugin>
-      <pose>0 0 0 0 0 0</pose>
-    </sensor>
-  </gazebo>
-  <!-- Lidar -->
-  <gazebo reference="lidar_link">
-    <sensor type="gpu_ray" name="RP_lidar">
-      <pose>0 0 0 0 0 0</pose>
-      <visualize>false</visualize>
-      <update_rate>${update_rate}</update_rate>
-      <ray>
-        <scan>
-          <horizontal>
-            <samples>720</samples>
-            <resolution>1</resolution>
-            <min_angle>-3.14159</min_angle>
-            <max_angle>3.14159</max_angle>
-          </horizontal>
-        </scan>
-        <range>
-          <min>0.15</min>
-          <max>6.0</max>
-          <resolution>0.5</resolution>
-        </range>
-        <noise>
-          <type>gaussian</type>
-          <!-- Noise parameters based on published spec for Hokuyo laser
-               achieving "+-30mm" accuracy at range < 10m.  A mean of 0.0m and
-               stddev of 0.01m will put 99.7% of samples within 0.03m of the true
-               reading. -->
-          <mean>0.0</mean>
-          <stddev>0.01</stddev>
-        </noise>
-      </ray>
-      <plugin name="gazebo_ros_head_hokuyo_controller" filename="libgazebo_ros_gpu_laser.so">
-        <topicName>/scan</topicName>
-        <frameName>lidar_link</frameName>
-      </plugin>
-    </sensor>
-  </gazebo>
 </robot>
